File: KitTen.brd (EAGLE design)
At the start: 68.6 x 53.3 mm, 33 parts, among them IC1 ATMEGA328P, Q1 2N7000, X1 16MHz HC49S

Commit message: Improved silkscreen, removed docs reference from README, bumped version for 2.1 release
Other:
- board text added: "v2.1"
- board text removed: "ROHS"
- board text removed: "v2.0"
Changed lines of the file:
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@@
 <wire x1="0.508" y1="50.8" x2="2.54" y2="52.832" width="0.3048" layer="22" curve="-90"/>
 <wire x1="0.508" y1="48.006" x2="0.508" y2="50.927" width="0.3048" layer="22"/>
-<wire x1="30.734" y1="26.67" x2="29.337" y2="25.273" width="0.5588" layer="22"/>
-<wire x1="29.337" y1="25.273" x2="26.797" y2="27.813" width="0.5588" layer="22"/>
 <wire x1="11.43" y1="46.99" x2="1.27" y2="46.99" width="0.4064" layer="21"/>
 <wire x1="1.27" y1="46.99" x2="1.27" y2="31.75" width="0.4064" layer="21"/>
@@
 <text x="25.019" y="30.607" size="1.6764" layer="21" font="vector" ratio="17" rot="R90">freetronics</text>
 <text x="1.778" y="49.911" size="2.1844" layer="21" font="vector" ratio="17">KitTen</text>
-<text x="7.62" y="48.5394" size="1.016" layer="21" font="vector" ratio="17">v2.0</text>
+<text x="7.62" y="48.5394" size="1.016" layer="21" font="vector" ratio="17">v2.1</text>
 <text x="41.529" y="47.244" size="0.9144" layer="21" font="vector" ratio="15">Digital</text>
 <text x="38.862" y="48.26" size="0.8128" layer="21" font="vector" ratio="15">9</text>
@@
 <text x="49.276" y="47.371" size="0.762" layer="22" font="vector" ratio="15" rot="MR0">PWM</text>
 <text x="2.286" y="13.208" size="1.1684" layer="21" font="vector" ratio="17">7-12VDC</text>
-<text x="30.988" y="23.368" size="1.27" layer="22" font="vector" ratio="17" rot="MR0">ROHS</text>
 <text x="1.905" y="32.512" size="0.8128" layer="21" font="vector" ratio="17">BLACK:GND</text>
 <text x="1.905" y="45.212" size="0.8128" layer="21" font="vector" ratio="17">GREEN:RTS</text>
@@
 <text x="1.905" y="42.672" size="0.8128" layer="21" font="vector" ratio="17">YELLOW:TX</text>
 <text x="11.938" y="49.911" size="2.1844" layer="22" font="vector" ratio="17" rot="MR0">KitTen</text>
-<text x="5.08" y="48.5394" size="1.016" layer="22" font="vector" ratio="17" rot="MR0">v2.0</text>
+<text x="5.08" y="48.5394" size="1.016" layer="22" font="vector" ratio="17" rot="MR0">v2.1</text>
 <text x="13.208" y="46.609" size="1.016" layer="21" font="vector" ratio="17">PWR SOURCE</text>
 <text x="14.224" y="45.466" size="1.016" layer="21" font="vector" ratio="17">SELECTION</text>
