File: KitTen.sch (EAGLE design)
At the start: 33 parts, among them IC1 ATMEGA328P, P5V M01SMD, Q1 2N7000, X1 16MHz HC49S

Commit message: Improved silkscreen, removed docs reference from README, bumped version for 2.1 release
Other:
- note added: "SKU: KITTEN"
- note added: "V2.1 (2014-09-01)"
- note removed: "SKU: FREE-KITTEN"
- note removed: "V2.0 (2013-02-14)"
Changed lines of the file:
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@@
 <?xml version="1.0" encoding="utf-8"?>
 <!DOCTYPE eagle SYSTEM "eagle.dtd">
-<eagle version="6.3">
+<eagle version="6.5.0">
 <drawing>
 <settings>
@@
 <text x="45.72" y="8.382" size="1.778" layer="94">Draw your project schematic here</text>
 <text x="147.32" y="12.7" size="3.048" layer="94">Freetronics KitTen</text>
-<text x="215.9" y="6.858" size="1.778" layer="94">V2.0 (2013-02-14)</text>
-<text x="187.706" y="6.858" size="1.778" layer="94">SKU: FREE-KITTEN</text>
+<text x="215.9" y="6.858" size="1.778" layer="94">V2.1 (2014-09-01)</text>
+<text x="187.706" y="6.858" size="1.778" layer="94">SKU: KITTEN</text>
 <text x="147.066" y="6.858" size="1.778" layer="94">www.freetronics.com/kitten</text>
 <text x="7.62" y="143.51" size="1.778" layer="94">DC Regulated Power Supply (optional)</text>
